Commit message: fixed robot model to include custom ee

File: path_planning/include/urdf/ur.urdf.xacro (robot description, xacro)
@@ -4,5 +4,5 @@
    <xacro:arg name="name" default="ur"/>
    <!-- import main macro -->
-   <xacro:include filename="$(find ur_description)/urdf/ur_macro.xacro"/>
+   <xacro:include filename="$(find ur3_bottle_sorter)/include/urdf/ur_macro.xacro"/>
    <!-- possible 'ur_type' values: ur3, ur3e, ur5, ur5e, ur10, ur10e, ur16e, ur20, ur30 -->
    <!-- the default value should raise an error in case this was called without defining the type -->

File: path_planning/include/urdf/ur_macro.xacro (robot description, xacro)
@@ -438,4 +438,24 @@
       <child link="${tf_prefix}tool0"/>
     </joint>
+    <!-- Custom End Effector Link -->
+    <link name="${tf_prefix}custom_ee_link">
+      <visual>
+        <origin xyz="0 0 0.05" rpy="0 0 0"/>
+        <geometry>
+          <mesh filename="package://ur3_bottle_sorter/include/meshes/endeffector/visual/ee.STL" scale="0.001 0.001 0.001"/>
+        </geometry>
+      </visual>
+      <collision>
+        <origin xyz="0 0 0.05" rpy="0 0 0"/>
+        <geometry>
+          <mesh filename="package://ur3_bottle_sorter/include/meshes/endeffector/collision/ee.STL" scale="0.001 0.001 0.001"/>
+        </geometry>
+      </collision>
+    </link>
+    <joint name="${tf_prefix}ee_mount" type="fixed">
+      <parent link="${tf_prefix}tool0"/>
+      <child link="${tf_prefix}custom_ee_link"/>
+      <origin xyz="-0.195 -0.222 0.202" rpy="-1.5708 0 0"/>
+    </joint>
   </xacro:macro>
 </robot>
